File: ISASTM.sch (KiCad schematic (older format))
At the start: 1 part, among them J1 Bus_ISA_16bit

Commit message: Add connector
Parts:
- removed J1: Bus_ISA_16bit, isastm:ISA16, symbol Connector:Bus_ISA_16bit
- added J1: Bus_ISA_8bit, ISASTM:Conn_Edge_PCB_ISA8, symbol Connector:Bus_ISA_8bit
Connections:
- net labels added: A0, A1, A10, A11, A12, A13, A14, A15, A16, A17, A18, A19, A2, A3, A4, A5, A6, A7, A8, A9, AEN, D0, D1, D2, D3, D4, D5, D6, D7, IO_CH_RDY, ~IO_CH_CK
- wire segments 32 -> 61
Changed lines of the file:
@@
 $EndDescr
 $Comp
-L Connector:Bus_ISA_16bit J1
-U 1 1 5F55CB3F
-P 2750 3950
-F 0 "J1" H 2750 6717 50  0000 C CNN
-F 1 "Bus_ISA_16bit" H 2750 6626 50  0000 C CNN
-F 2 "isastm:ISA16" H 2750 4000 50  0001 C CNN
-F 3 "https://en.wikipedia.org/wiki/Industry_Standard_Architecture" H 2750 4000 50  0001 C CNN
-	1    2750 3950
-	1    0    0    -1
-$EndComp
-$Comp
-L power:GND #PWR?
-U 1 1 5F5604B9
-P 1850 6350
-F 0 "#PWR?" H 1850 6100 50  0001 C CNN
-F 1 "GND" H 1700 6300 50  0000 C CNN
-F 2 "" H 1850 6350 50  0001 C CNN
-F 3 "" H 1850 6350 50  0001 C CNN
-	1    1850 6350
-	1    0    0    -1
-$EndComp
-$Comp
-L power:GND #PWR?
+L power:GND #PWR08
 U 1 1 5F561F50
 P 1850 4450
-F 0 "#PWR?" H 1850 4200 50  0001 C CNN
+F 0 "#PWR08" H 1850 4200 50  0001 C CNN
 F 1 "GND" H 1700 4400 50  0000 C CNN
 F 2 "" H 1850 4450 50  0001 C CNN
@@
 $EndComp
 $Comp
-L power:GND #PWR?
+L power:GND #PWR05
 U 1 1 5F56224F
 P 1500 2350
-F 0 "#PWR?" H 1500 2100 50  0001 C CNN
+F 0 "#PWR05" H 1500 2100 50  0001 C CNN
 F 1 "GND" H 1505 2177 50  0000 C CNN
 F 2 "" H 1500 2350 50  0001 C CNN
@@
 $EndComp
 $Comp
-L power:GND #PWR?
+L power:GND #PWR07
 U 1 1 5F562491
 P 1600 1450
-F 0 "#PWR?" H 1600 1200 50  0001 C CNN
+F 0 "#PWR07" H 1600 1200 50  0001 C CNN
 F 1 "GND" H 1600 1500 50  0000 C CNN
 F 2 "" H 1600 1450 50  0001 C CNN
@@
 Wire Wire Line
 	1850 4450 2050 4450
-Wire Wire Line
-	1850 6350 2050 6350
-$Comp
-L power:+5V #PWR?
-U 1 1 5F563770
-P 1850 6150
-F 0 "#PWR?" H 1850 6000 50  0001 C CNN
-F 1 "+5V" H 1700 6200 50  0000 C CNN
-F 2 "" H 1850 6150 50  0001 C CNN
-F 3 "" H 1850 6150 50  0001 C CNN
-	1    1850 6150
-	1    0    0    -1
-$EndComp
-$Comp
-L power:+5V #PWR?
+$Comp
+L power:+5V #PWR01
 U 1 1 5F564A3C
 P 1500 1650
-F 0 "#PWR?" H 1500 1500 50  0001 C CNN
+F 0 "#PWR01" H 1500 1500 50  0001 C CNN
 F 1 "+5V" H 1300 1700 50  0000 C CNN
 F 2 "" H 1500 1650 50  0001 C CNN
@@
 	1    0    0    -1
 $EndComp
-Wire Wire Line
-	1850 6150 2050 6150
-$Comp
-L power:-5V #PWR?
+$Comp
+L power:-5V #PWR02
 U 1 1 5F565103
 P 1500 1850
-F 0 "#PWR?" H 1500 1950 50  0001 C CNN
+F 0 "#PWR02" H 1500 1950 50  0001 C CNN
 F 1 "-5V" H 1300 1900 50  0000 C CNN
 F 2 "" H 1500 1850 50  0001 C CNN
@@
 	1500 1850 2050 1850
 $Comp
-L power:-12V #PWR?
+L power:-12V #PWR03
 U 1 1 5F5660B6
 P 1500 2050
-F 0 "#PWR?" H 1500 2150 50  0001 C CNN
+F 0 "#PWR03" H 1500 2150 50  0001 C CNN
 F 1 "-12V" H 1300 2100 50  0000 C CNN
 F 2 "" H 1500 2050 50  0001 C CNN
@@
 $EndComp
 $Comp
-L power:+12V #PWR?
+L power:+12V #PWR04
 U 1 1 5F566E3C
 P 1500 2250
-F 0 "#PWR?" H 1500 2100 50  0001 C CNN
+F 0 "#PWR04" H 1500 2100 50  0001 C CNN
 F 1 "+12V" H 1300 2300 50  0000 C CNN
 F 2 "" H 1500 2250 50  0001 C CNN
@@
 ALE
 $Comp
-L power:+5V #PWR?
+L power:+5V #PWR06
 U 1 1 5F570D10
 P 1500 4250
-F 0 "#PWR?" H 1500 4100 50  0001 C CNN
+F 0 "#PWR06" H 1500 4100 50  0001 C CNN
 F 1 "+5V" H 1300 4300 50  0000 C CNN
 F 2 "" H 1500 4250 50  0001 C CNN
@@
 Wire Wire Line
 	2050 3350 1650 3350
+$Comp
+L Connector:Bus_ISA_8bit J1
+U 1 1 5F5E82DF
+P 2750 2950
+F 0 "J1" H 2750 4717 50  0000 C CNN
+F 1 "Bus_ISA_8bit" H 2750 4626 50  0000 C CNN
+F 2 "ISASTM:Conn_Edge_PCB_ISA8" H 2750 2950 50  0001 C CNN
+F 3 "https://en.wikipedia.org/wiki/Industry_Standard_Architecture" H 2750 2950 50  0001 C CNN
+	1    2750 2950
+	1    0    0    -1
+$EndComp
+Text Label 3900 1450 2    50   ~ 0
+~IO_CH_CK
+Wire Wire Line
+	3450 1450 3900 1450
+Text Label 3900 1550 2    50   ~ 0
+D7
+Text Label 3900 1650 2    50   ~ 0
+D6
+Text Label 3900 1750 2    50   ~ 0
+D5
+Text Label 3900 1850 2    50   ~ 0
+D4
+Text Label 3900 1950 2    50   ~ 0
+D3
+Text Label 3900 2050 2    50   ~ 0
+D2
+Text Label 3900 2150 2    50   ~ 0
+D1
+Text Label 3900 2250 2    50   ~ 0
+D0
+Text Label 3900 2350 2    50   ~ 0
+IO_CH_RDY
+Text Label 3900 2450 2    50   ~ 0
+AEN
+Text Label 3900 2550 2    50   ~ 0
+A19
+Text Label 3900 2650 2    50   ~ 0
+A18
+Text Label 3900 2750 2    50   ~ 0
+A17
+Text Label 3900 2850 2    50   ~ 0
+A16
+Text Label 3900 2950 2    50   ~ 0
+A15
+Text Label 3900 3050 2    50   ~ 0
+A14
+Text Label 3900 3150 2    50   ~ 0
+A13
+Text Label 3900 3250 2    50   ~ 0
+A12
+Text Label 3900 3350 2    50   ~ 0
+A11
+Text Label 3900 3450 2    50   ~ 0
+A10
+Text Label 3900 3550 2    50   ~ 0
+A9
+Text Label 3900 3650 2    50   ~ 0
+A8
+Text Label 3900 3750 2    50   ~ 0
+A7
+Text Label 3900 3850 2    50   ~ 0
+A6
+Text Label 3900 3950 2    50   ~ 0
+A5
+Text Label 3900 4050 2    50   ~ 0
+A4
+Text Label 3900 4150 2    50   ~ 0
+A3
+Text Label 3900 4250 2    50   ~ 0
+A2
+Text Label 3900 4350 2    50   ~ 0
+A1
+Text Label 3900 4450 2    50   ~ 0
+A0
+Wire Wire Line
+	3900 4450 3450 4450
+Wire Wire Line
+	3450 4350 3900 4350
+Wire Wire Line
+	3900 4250 3450 4250
+Wire Wire Line
+	3450 4150 3900 4150
+Wire Wire Line
+	3900 4050 3450 4050
+Wire Wire Line
+	3450 3950 3900 3950
+Wire Wire Line
+	3900 3850 3450 3850
+Wire Wire Line
+	3450 3750 3900 3750
+Wire Wire Line
+	3900 3650 3450 3650
+Wire Wire Line
+	3450 3550 3900 3550
+Wire Wire Line
+	3900 3450 3450 3450
+Wire Wire Line
+	3450 3350 3900 3350
+Wire Wire Line
+	3900 3250 3450 3250
+Wire Wire Line
+	3450 3150 3900 3150
+Wire Wire Line
+	3900 3050 3450 3050
+Wire Wire Line
+	3450 2950 3900 2950
+Wire Wire Line
+	3450 2850 3900 2850
+Wire Wire Line
+	3450 2750 3900 2750
+Wire Wire Line
+	3900 2650 3450 2650
+Wire Wire Line
+	3450 2550 3900 2550
+Wire Wire Line
+	3900 2450 3450 2450
+Wire Wire Line
+	3450 2350 3900 2350
+Wire Wire Line
+	3900 2250 3450 2250
+Wire Wire Line
+	3450 2150 3900 2150
+Wire Wire Line
+	3900 2050 3450 2050
+Wire Wire Line
+	3450 1950 3900 1950
+Wire Wire Line
+	3900 1850 3450 1850
+Wire Wire Line
+	3450 1750 3900 1750
+Wire Wire Line
+	3900 1650 3450 1650
+Wire Wire Line
+	3450 1550 3900 1550
 $EndSCHEMATC

Commit message: Add ISA bus, level shifters, memory pinout
Parts:
- added C1, C2: 2.2u, Capacitor_SMD:C_0603_1608Metric, symbol Device:C
- added C12, C13, C14, C15, C16, C17, C19, C20, C21, C22, C23, C24, C25, C26, C27, C28, C29, C30, C31, C32, C35, C36, C37: 100n, Capacitor_SMD:C_0402_1005Metric, symbol Device:C
- added C18: 10u, Capacitor_SMD:C_0603_1608Metric, symbol Device:C
- added C33, C7: 1u, Capacitor_SMD:C_0402_1005Metric, symbol Device:C
- added C34: 22u, Capacitor_SMD:C_0603_1608Metric, symbol Device:C
- added C5, C6: 20p, Capacitor_SMD:C_0402_1005Metric, symbol Device:C
- added J3: Boot select, Connector_PinHeader_2.54mm:PinHeader_1x03_P2.54mm_Vertical, symbol Connector_Generic:Conn_01x03
- added R1, R10, R11, R12, R3, R4, R5, R6, R7, R9: 10k, Resistor_SMD:R_0402_1005Metric, symbol Device:R
- added R2: 10R, Resistor_SMD:R_0402_1005Metric, symbol Device:R
- added R8: 100k, Resistor_SMD:R_0402_1005Metric, symbol Device:R
- added SW1: Reset, CMM2-JLC:TS-1187A-X-X-X, symbol Switch:SW_Push
- added U1: STM32H743IITx, Package_QFP:LQFP-176_24x24mm_P0.5mm, symbol MCU_ST_STM32H7:STM32H743IITx
- added U10, U11, U12, U13, U3, U4, U6, U7, U8, U9: SN74AVC8T245PW, Package_SO:TSSOP-24_4.4x7.8mm_P0.65mm, symbol Logic_LevelTranslator:SN74AVC8T245PW
- added U2: MT48LC16M16A2P, Package_SO:TSOP-II-54_22.2x10.16mm_P0.8mm, symbol SDRAM_Micron:MT48LC16M16A2
- added U5: AMS1117-3.3, Package_TO_SOT_SMD:SOT-223-3_TabPin2, symbol Regulator_Linear:AMS1117-3.3
- added U?: USB3343, Package_DFN_QFN:QFN-24-1EP_4x4mm_P0.5mm_EP2.6x2.6mm, symbol Interface_USB:USB3343
- added X1: SG-7050CAN, Oscillator:Oscillator_SMD_SeikoEpson_SG8002CA-4Pin_7.0x5.0mm, symbol Oscillator:SG-7050CAN
- added Y2: 8 MHz, Crystal:Crystal_SMD_5032-2Pin_5.0x3.2mm, symbol Device:Crystal
Connections:
- net +5V: now also C18.1, C22.1, R10.2, R11.2, R12.2, R3.2, R4.2, R5.2, R6.2, R9.2, U10.1 (VCCA), U11.1 (VCCA), U12.1 (VCCA), U13.1 (VCCA), U3.1 (VCCA), U4.1 (VCCA), U5.3 (VI), U6.1 (VCCA), U7.1 (VCCA), U8.1 (VCCA), U9.1 (VCCA)
- net A0: now also U9.3 (A1)
- net A1: now also U9.4 (A2)
- net A10: now also U10.5 (A3)
- net A11: now also U10.6 (A4)
- net A12: now also U10.7 (A5)
- net A13: now also U10.8 (A6)
- net A14: now also U10.9 (A7)
- net A15: now also U10.10 (A8)
- net A16: now also U11.3 (A1)
- net A17: now also U11.4 (A2)
- net A18: now also U11.5 (A3)
- net A19: now also U11.6 (A4)
- net A2: now also U9.5 (A3)
- net A3: now also U9.6 (A4)
- net A4: now also U9.7 (A5)
- net A5: now also U9.8 (A6)
- net A6: now also U9.9 (A7)
- net A7: now also U9.10 (A8)
- net A8: now also U10.3 (A1)
- net A9: now also U10.4 (A2)
- net AEN: now also U4.7 (A5)
- net ALE: now also U4.8 (A6)
- net D0: now also R3.1, U3.3 (A1)
- net D1: now also R4.1, U3.4 (A2)
- net D2: now also R5.1, U3.5 (A3)
- net D3: now also R6.1, U3.6 (A4)
- net D4: now also R9.1, U3.7 (A5)
- net D5: now also R10.1, U3.8 (A6)
- net D6: now also R11.1, U3.9 (A7)
- net D7: now also R12.1, U3.10 (A8)
- net DRQ1: now also U7.3 (A1)
- net DRQ2: now also U7.4 (A2)
- net DRQ3: now also U7.5 (A3)
- net GND: now also C1.2, C12.2, C13.2, C14.2, C15.2, C16.2, C17.2, C18.2, C19.2, C2.1, C20.2, C21.2, C22.2, C23.2, C24.2, C25.2, C26.2, C27.2, C28.2, C29.2, C30.2, C31.2, C32.2, C33.2, C34.2, C35.2, C36.2, C37.2, C5.1, C6.2, C7.2, J3.3 (Pin_3), SW1.1, U1.102 (VSS), U1.113 (VSS), U1.126 (VSS), U1.135 (VSS), U1.14 (VSS), U1.148 (VSS), U1.158 (VSS), U1.22 (VSS), U1.37 (VSSA), U1.48 (VSS), U1.61 (VSS), U1.71 (VSS), U1.90 (VSS), U10.11 (GND), U10.12 (GND), U10.13 (GND), U11.11 (GND), U11.12 (GND), U11.13 (GND), U12.11 (GND), U12.12 (GND), U12.13 (GND), U13.11 (GND), U13.12 (GND), U13.13 (GND), U2.12 (VSSQ), U2.28 (VSS), U2.41 (VSS), U2.46 (VSSQ), U2.52 (VSSQ), U2.54 (VSS), U2.6 (VSSQ), U3.11 (GND), U3.12 (GND), U3.13 (GND), U4.11 (GND), U4.12 (GND), U4.13 (GND), U5.1 (GND), U6.11 (GND), U6.12 (GND), U6.13 (GND), U7.11 (GND), U7.12 (GND), U7.13 (GND), U8.11 (GND), U8.12 (GND), U8.13 (GND), U9.11 (GND), U9.12 (GND), U9.13 (GND), X1.2 (GND)
- net IO_CH_RDY: now also U6.3 (A1)
- net IRQ2: now also U6.4 (A2)
- net IRQ3: now also U6.5 (A3)
- net IRQ4: now also U6.6 (A4)
- net IRQ5: now also U6.7 (A5)
- net IRQ6: now also U6.8 (A6)
- net IRQ7: now also U6.9 (A7)
- net OSC: now also U11.10 (A8)
- net RESET: now also C33.1, R8.1, SW1.2, U1.31 (NRST); no longer J1.2 (RESET)
- net ~DACK1: now also U12.3 (A1)
- net ~DACK2: now also U12.4 (A2)
- net ~DACK3: now also U12.5 (A3)
- net ~IOR: now also U4.6 (A4)
- net ~IOW: now also U4.5 (A3)
- net ~IO_CH_CK: now also U6.10 (A8)
- net ~REFRESH: now also U4.9 (A7)
- net ~SMEMR: now also U4.4 (A2)
- net ~SMEMW: now also U4.3 (A1)
- new net: C2.2, U1.125 (VCAP2)
- new net: R1.1, U1.171 (PDR_ON)
- new net: C6.1, U1.29 (PH0), Y2.2
- new net: C5.2, U1.30 (PH1), Y2.1
- new net: C7.1, R2.2, U1.38 (VREF+)
- new net: C1.1, U1.81 (VCAP1)
- new net: J3.2 (Pin_2), R7.1
- new net: U11.14 (B8), X1.3 (OUT)
- new net +3V3: C12.1, C13.1, C14.1, C15.1, C16.1, C17.1, C19.1, C20.1, C21.1, C23.1, C24.1, C25.1, C26.1, C27.1, C28.1, C29.1, C30.1, C31.1, C32.1, C34.1, C35.1, C36.1, C37.1, J3.1 (Pin_1), R1.2, R2.1, R8.2, U1.103 (VDD), U1.114 (VDD33_USB), U1.127 (VDD), U1.136 (VDD), U1.149 (VDD), U1.15 (VDD), U1.159 (VDD), U1.172 (VDD), U1.23 (VDD), U1.36 (VDD), U1.39 (VDDA), U1.49 (VDD), U1.62 (VDD), U1.72 (VDD), U1.82 (VDD), U1.91 (VDD), U10.23 (VCCB), U10.24 (VCCB), U11.23 (VCCB), U11.24 (VCCB), U12.23 (VCCB), U12.24 (VCCB), U13.23 (VCCB), U13.24 (VCCB), U2.1 (VDD), U2.14 (VDD), U2.27 (VDD), U2.3 (VDDQ), U2.43 (VDDQ), U2.49 (VDDQ), U2.9 (VDDQ), U3.23 (VCCB), U3.24 (VCCB), U4.23 (VCCB), U4.24 (VCCB), U5.2 (VO), U6.23 (VCCB), U6.24 (VCCB), U7.23 (VCCB), U7.24 (VCCB), U8.23 (VCCB), U8.24 (VCCB), U9.23 (VCCB), U9.24 (VCCB), X1.1 (~ST), X1.4 (VCC)
- new net ADDRESS_DIR: U10.2 (DIR), U11.2 (DIR), U9.2 (DIR)
- new net ADDRESS_OE: U10.22 (~OE), U11.22 (~OE), U9.22 (~OE)
- new net BOOT0: R7.2, U1.166 (BOOT0)
- new net CONTROL1_DIR: U4.2 (DIR)
- new net CONTROL1_OE: U4.22 (~OE)
- new net CONTROL2_DIR: U7.2 (DIR)
- new net CONTROL2_OE: U7.22 (~OE)
- new net CONTROL3_DIR: U12.2 (DIR)
- new net CONTROL3_OE: U12.22 (~OE)
- new net DATA_DIR: U3.2 (DIR)
- new net DATA_OE: U3.22 (~OE)
- new net IRQ_DIR: U6.2 (DIR)
- new net IRQ_OE: U6.22 (~OE)
- new net ISARESET: J1.2 (RESET), U4.10 (A8)
- new net MEM_PD0: U1.142 (PD0), U2.5 (DQ2)
- new net MEM_PD1: U1.143 (PD1), U2.7 (DQ3)
- new net MEM_PD10: U1.98 (PD10), U2.53 (DQ15)
- new net MEM_PD14: U1.104 (PD14), U2.2 (DQ0)
- new net MEM_PD15: U1.105 (PD15), U2.4 (DQ1)
- new net MEM_PD8: U1.96 (PD8), U2.50 (DQ13)
- new net MEM_PD9: U1.97 (PD9), U2.51 (DQ14)
- new net MEM_PE0: U1.169 (PE0), U2.15 (DQML)
- new net MEM_PE1: U1.170 (PE1), U2.39 (DQMH)
- new net MEM_PE10: U1.73 (PE10), U2.13 (DQ7)
- new net MEM_PE11: U1.74 (PE11), U2.42 (DQ8)
- new net MEM_PE12: U1.75 (PE12), U2.44 (DQ9)
- new net MEM_PE13: U1.76 (PE13), U2.45 (DQ10)
- new net MEM_PE14: U1.77 (PE14), U2.47 (DQ11)
- new net MEM_PE15: U1.78 (PE15), U2.48 (DQ12)
- new net MEM_PE7: U1.68 (PE7), U2.8 (DQ4)
- new net MEM_PE8: U1.69 (PE8), U2.10 (DQ5)
- new net MEM_PE9: U1.70 (PE9), U2.11 (DQ6)
- new net MEM_PF0: U1.16 (PF0), U2.23 (A0)
- new net MEM_PF1: U1.17 (PF1), U2.24 (A1)
- new net MEM_PF11: U1.59 (PF11), U2.18 (~RAS~)
- new net MEM_PF12: U1.60 (PF12), U2.31 (A6)
- new net MEM_PF13: U1.63 (PF13), U2.32 (A7)
- new net MEM_PF14: U1.64 (PF14), U2.33 (A8)
- new net MEM_PF15: U1.65 (PF15), U2.34 (A9)
- new net MEM_PF2: U1.18 (PF2), U2.25 (A2)
- new net MEM_PF3: U1.19 (PF3), U2.26 (A3)
- new net MEM_PF4: U1.20 (PF4), U2.29 (A4)
- new net MEM_PF5: U1.21 (PF5), U2.30 (A5)
- new net MEM_PG0: U1.66 (PG0), U2.22 (A10)
- new net MEM_PG1: U1.67 (PG1), U2.35 (A11)
- new net MEM_PG15: U1.160 (PG15), U2.17 (~CAS~)
- new net MEM_PG2: U1.106 (PG2), U2.36 (A12)
- new net MEM_PG4: U1.108 (PG4), U2.20 (BA0)
- new net MEM_PG5: U1.109 (PG5), U2.21 (BA1)
- new net MEM_PG8: U1.112 (PG8), U2.38 (CLK)
- new net MEM_PH5: U1.46 (PH5), U2.16 (~WE~)
- new net MEM_PH6: U1.83 (PH6), U2.19 (~CS~)
- new net MEM_PH7: U1.84 (PH7), U2.37 (CKE)
- new net SPARE1_DIR: U8.2 (DIR)
- new net SPARE1_OE: U8.22 (~OE)
- new net SPARE2_DIR: U13.2 (DIR)
- new net SPARE2_OE: U13.22 (~OE)
- new net USB_HOST_D+: U1.123 (PA12)
- new net USB_HOST_D-: U1.122 (PA11)
- new net VBAT: U1.6 (VBAT)
Other:
- note added: "CPU"
- note added: "Interruptleitungen brauchen vermutlich PullUps? \nRefresh-Leitung braucht Pullup (und ist theoretisch bidirektional)\nPrüfen ob Adressleitungen nie geschaltet werden müssen (weil der Oszillator da dranhängt)\n\nDIR/OE Pins brauchen Pull Ups/Downs für eine sinnvolle Default-Config\n\nDMA-Pins\nSteuerleitungen\n14. MHz OSC\n\nUSB 1.1\nTagconnect\n"
- note added: "SDRAM"
- moved on the sheet: J1

Commit message: Add USB PHY, USB connectors, pull ups, DRQ/IRQ
Parts:
- added C? (x2): 6.8pF, Capacitor_SMD:C_0402_1005Metric, symbol Device:C
- added C? (x3): 1u, Capacitor_SMD:C_0402_1005Metric, symbol Device:C
- added C? (x3): 100n, Capacitor_SMD:C_0402_1005Metric, symbol Device:C
- added J? (x2): USB_C_Receptacle_USB2.0, Connector_USB:USB_C_Receptacle_Palconn_UTC16-G, symbol Connector:USB_C_Receptacle_USB2.0
- added J?: TagConnect_TC2030_SWD, Connector:Tag-Connect_TC2030-IDC-NL_2x03_P1.27mm_Vertical, symbol Connector_TagConnect:TagConnect_TC2030_SWD
- added JP?: SolderJumper_2_Open, symbol Jumper:SolderJumper_2_Open
- added R?: 1M, Resistor_SMD:R_0402_1005Metric, symbol Device:R
- added R?: 7.5k, Resistor_SMD:R_0402_1005Metric, symbol Device:R
- added R?: 560R, Resistor_SMD:R_0603_1608Metric, symbol Device:R
- added R? (x4): 5.1k, Resistor_SMD:R_0402_1005Metric, symbol Device:R
- added R?: 20k, Resistor_SMD:R_0402_1005Metric, symbol Device:R
- added R? (x17): 100k, Resistor_SMD:R_0402_1005Metric, symbol Device:R
- added R?: 1k, Resistor_SMD:R_0402_1005Metric, symbol Device:R
- added R? (x5): 4.7k, Resistor_SMD:R_0402_1005Metric, symbol Device:R
- added U?: SRV05-4, Package_TO_SOT_SMD:SOT-23-6, symbol Power_Protection:SRV05-4
- added Y?: 26 MHz, Crystal:Crystal_SMD_3225-4Pin_3.2x2.5mm, symbol Device:Crystal_GND24_Small
Connections:
- net RESET is gone; now on net ~RESET: C33.1, R8.1, SW1.2, U1.31 (NRST)
- net +3V3: now also U?.9 (VDDIO), C?.1, C?.2, J?.1 (VTGT), R?.1, R?.1, R?.1, R?.1, R?.1, R?.1, R?.1, R?.1
- net +5V: now also U?.16 (VBAT), C?.2, JP?.2 (B), R?.1, R?.1, R?.1, R?.1, R?.1, R?.1
- net CLK: now also U12.7 (A5)
- net DRQ1: now also R?.2
- net DRQ2: now also R?.2
- net DRQ3: now also R?.2
- net GND: now also U11.10 (A8), U11.14 (B8), U11.15 (B7), U11.16 (B6), U11.17 (B5), U11.7 (A5), U11.8 (A6), U11.9 (A7), U12.10 (A8), U12.14 (B8), U4.10 (A8), U4.14 (B8), U7.10 (A8), U7.14 (B8), U7.15 (B7), U7.16 (B6), U7.17 (B5), U7.18 (B4), U7.6 (A4), U7.7 (A5), U7.8 (A6), U7.9 (A7), U?.25 (GND), C?.1, C?.1, C?.1, C?.1, C?.2, C?.2, C?.2, C?.2, J?.5 (GND), J?.A1 (GND), J?.A1 (GND), J?.A12 (GND), J?.A12 (GND), J?.B1 (GND), J?.B1 (GND), J?.B12 (GND), J?.B12 (GND), J?.S1 (SHIELD), J?.S1 (SHIELD), R?.1, R?.1, R?.1, R?.1, R?.1, R?.1, R?.1, R?.1, R?.1, R?.1, R?.1, R?.2, R?.2, R?.2, U?.2 (VN), Y?.2, Y?.4
- net IO_CH_RDY: now also R?.2
- net IRQ2: now also R?.2
- net IRQ3: now also R?.2
- net IRQ4: now also R?.2
- net IRQ5: now also R?.2
- net IRQ6: now also R?.2
- net IRQ7: now also R?.2
- net ISARESET: now also U4.9 (A7); no longer U4.10 (A8)
- net OSC: now also U12.9 (A7); no longer U11.10 (A8)
- net TC: now also U12.6 (A4)
- net ~IOR: now also R?.2
- net ~IOW: now also R?.2
- net ~IO_CH_CK: now also R?.2
- net ~REFRESH: now also U1.162 (PB4); no longer U4.9 (A7)
- net ~SMEMR: now also R?.2
- net ~SMEMW: now also R?.2
- net ~NOWS: now reaches J1.8 (UNUSED)
- net ~NOWS: now also U12.8 (A6)
- net LV_A7: now reaches U9.14 (B8)
- net LV_A7: now also U1.130 (PH15)
- net LV_A6: now reaches U9.15 (B7)
- net LV_A6: now also U1.129 (PH14)
- net LV_A5: now reaches U9.16 (B6)
- net LV_A5: now also U1.128 (PH13)
- net LV_A4: now reaches U9.17 (B5)
- net LV_A4: now also U1.89 (PH12)
- net LV_A3: now reaches U9.18 (B4)
- net LV_A3: now also U1.88 (PH11)
- net LV_A2: now reaches U9.19 (B3)
- net LV_A2: now also U1.87 (PH10)
- net LV_A1: now reaches U9.20 (B2)
- net LV_A1: now also U1.86 (PH9)
- net LV_A0: now reaches U9.21 (B1)
- net LV_A0: now also U1.85 (PH8)
- net SWDIO: now reaches U1.124 (PA13)
- net SWDIO: now also J?.2 (SWDIO)
- net LV_D0: now reaches U1.131 (PI0)
- net LV_D0: now also U3.21 (B1)
- net LV_D1: now reaches U1.132 (PI1)
- net LV_D1: now also U3.20 (B2)
- net LV_D2: now reaches U1.133 (PI2)
- net LV_D2: now also U3.19 (B3)
- net LV_D3: now reaches U1.134 (PI3)
- net LV_D3: now also U3.18 (B4)
- net SWCLK: now reaches U1.137 (PA14)
- net SWCLK: now also J?.4 (SWCLK)
- net SWO: now reaches U1.161 (PB3)
- net SWO: now also J?.6 (SWO)
- net OTG_HS_ULPI_D7: now reaches U1.163 (PB5)
- net OTG_HS_ULPI_D7: now also U?.12 (DATA7)
- net LV_D4: now reaches U1.173 (PI4)
- net LV_D4: now also U3.17 (B5)
- net LV_D5: now reaches U1.174 (PI5)
- net LV_D5: now also U3.16 (B6)
- net LV_D6: now reaches U1.175 (PI6)
- net LV_D6: now also U3.15 (B7)
- net LV_D7: now reaches U1.176 (PI7)
- net LV_D7: now also U3.14 (B8)
- net OTG_HS_ULPI_STP: now reaches U1.32 (PC0)
- net OTG_HS_ULPI_STP: now also U?.24 (STP)
- net OTG_HS_ULPI_DIR: now reaches U1.34 (PC2_C)
- net OTG_HS_ULPI_DIR: now also U?.1 (DIR)
- net OTG_HS_ULPI_NXT: now reaches U1.35 (PC3_C)
- net OTG_HS_ULPI_NXT: now also U?.3 (NXT)
- net OTG_HS_ULPI_D0: now reaches U1.47 (PA3)
- net OTG_HS_ULPI_D0: now also U?.4 (DATA0)
- net OTG_HS_ULPI_CK: now reaches U1.51 (PA5)
- net OTG_HS_ULPI_CK: now also U?.2 (CLKOUT)
- net OTG_HS_ULPI_D1: now reaches U1.56 (PB0)
- net OTG_HS_ULPI_D1: now also U?.5 (DATA1)
- net OTG_HS_ULPI_D2: now reaches U1.57 (PB1)
- net OTG_HS_ULPI_D2: now also U?.6 (DATA2)
- net OTG_HS_ULPI_D3: now reaches U1.79 (PB10)
- net OTG_HS_ULPI_D3: now also U?.7 (DATA3)
- net OTG_HS_ULPI_D4: now reaches U1.80 (PB11)
- net OTG_HS_ULPI_D4: now also U?.8 (DATA4)
- net OTG_HS_ULPI_D5: now reaches U1.92 (PB12)
- net OTG_HS_ULPI_D5: now also U?.10 (DATA5)
- net OTG_HS_ULPI_D6: now reaches U1.93 (PB13)
- net OTG_HS_ULPI_D6: now also U?.11 (DATA6)
- net LV_ISARESET: now reaches U4.15 (B7)
- net LV_ALE: now reaches U4.16 (B6)
- net LV_AEN: now reaches U4.17 (B5)
- net ~LV_IOR: now reaches U4.18 (B4)
- net ~LV_IOW: now reaches U4.19 (B3)
- net ~LV_SMEMR: now reaches U4.20 (B2)
- net ~LV_SMEMW: now reaches U4.21 (B1)
- net LV_A15: now reaches U10.14 (B8)
- net LV_A14: now reaches U10.15 (B7)
- net LV_A13: now reaches U10.16 (B6)
- net LV_A12: now reaches U10.17 (B5)
- net LV_A11: now reaches U10.18 (B4)
- net LV_A10: now reaches U10.19 (B3)
- net LV_A9: now reaches U10.20 (B2)
- net LV_A8: now reaches U10.21 (B1)
- net at X1.3 (OUT): now also U12.15 (B7); no longer U11.14 (B8)
- net LV_A19: now reaches U11.18 (B4)
- net LV_A18: now reaches U11.19 (B3)
- net LV_A17: now reaches U11.20 (B2)
- net LV_A16: now reaches U11.21 (B1)
- net ~LV_IO_CH_CK: now reaches U6.14 (B8)
- net LV_IRQ7: now reaches U6.15 (B7)
- net LV_IRQ6: now reaches U6.16 (B6)
- net LV_IRQ5: now reaches U6.17 (B5)
- net LV_IRQ4: now reaches U6.18 (B4)
- net LV_IRQ3: now reaches U6.19 (B3)
- net LV_IRQ2: now reaches U6.20 (B2)
- net LV_IO_CH_RDY: now reaches U6.21 (B1)
- net LV_DRQ3: now reaches U7.19 (B3)
- net LV_DRQ2: now reaches U7.20 (B2)
- net LV_DRQ1: now reaches U7.21 (B1)
- net ~LV_NOWS: now reaches U12.16 (B6)
- net LV_CLK: now reaches U12.17 (B5)
- net LV_TC: now reaches U12.18 (B4)
- net ~LV_DACK3: now reaches U12.19 (B3)
- net ~LV_DACK2: now reaches U12.20 (B2)
- net ~LV_DACK1: now reaches U12.21 (B1)
- net at U?.13 (DP): now also J?.A6 (D+), J?.B6 (D+)
- net at U?.14 (DM): now also J?.A7 (D-), J?.B7 (D-)
- net at U?.15 (VDD33): now also U?.18 (ID), C?.2
- net at U?.17 (VBUS): now also R?.1
- net at U?.19 (RBIAS): now also R?.1
- net at U?.20 (XO): now also C?.1, R?.2, Y?.1
- net at U?.21 (REFCLK/XI): now also C?.1, R?.1, Y?.3
- net ~RESET: now reaches U?.22 (~RESETB)
- net ~RESET: now also J?.3 (~RESET)
- net at U?.23 (VDD18): now also C?.2
- net ADDRESS_OE renamed ~ADDRESS_OE
- net ~ADDRESS_OE: now also R?.2
- net CONTROL1_OE renamed ~CONTROL1_OE
- net ~CONTROL1_OE: now also R?.2
- net CONTROL2_OE renamed ~CONTROL2_OE
- net ~CONTROL2_OE: now also R?.2
- net CONTROL3_OE renamed ~CONTROL3_OE
- net ~CONTROL3_OE: now also R?.2
- net DATA_OE renamed ~DATA_OE
- net ~DATA_OE: now also R?.2
- net IRQ_OE renamed ~IRQ_OE
- net ~IRQ_OE: now also R?.2
- net SPARE1_OE renamed ~SPARE1_OE
- net ~SPARE1_OE: now also R?.2
- net SPARE2_OE renamed ~SPARE2_OE
- net ~SPARE2_OE: now also R?.2
- net USB_HOST_D+ renamed USB_FS_D+
- net USB_FS_D+: now also J?.A6 (D+), J?.B6 (D+), U?.3 (IO2)
- net USB_HOST_D- renamed USB_FS_D-
- net USB_FS_D-: now also J?.A7 (D-), J?.B7 (D-), U?.1 (IO1)
- new net: R?.1, R?.2
- new net: C?.1, J?.A4 (VBUS), J?.A9 (VBUS), J?.B4 (VBUS), J?.B9 (VBUS), R?.2
- new net: J?.A5 (CC1), R?.2 (x2)
- new net: J?.B5 (CC2), R?.1 (x2)
- new net: J?.A4 (VBUS), J?.A9 (VBUS), J?.B4 (VBUS), J?.B9 (VBUS), JP?.1 (A), U?.5 (VP)
- no-connect marks 1 -> 6
Other:
- note added: "Refresh-Leitung braucht Pullup (und ist theoretisch bidirektional)\n"
- note removed: "Interruptleitungen brauchen vermutlich PullUps? \nRefresh-Leitung braucht Pullup (und ist theoretisch bidirektional)\nPrüfen ob Adressleitungen nie geschaltet werden müssen (weil der Oszillator da dranhängt)\n\nDIR/OE Pins brauchen Pull Ups/Downs für eine sinnvolle Default-Config\n\nDMA-Pins\nSteuerleitungen\n14. MHz OSC\n\nUSB 1.1\nTagconnect\n"
- moved on the sheet: C1, C2, C5, C6, C7, R1, R2, U1, U2, U?, X1, Y2

Commit message: Add more decoupling
Parts:
- added C40, C41, C42, C43, C44, C45, C46, C47, C48, C49, C50, C51, C52, C53, C54, C55, C56, C57, C58, C59: 100n, Capacitor_SMD:C_0402_1005Metric, symbol Device:C
- added D1: White, LED_SMD:LED_0603_1608Metric, symbol Device:LED
- added D2: Red, LED_SMD:LED_0603_1608Metric, symbol Device:LED
- added D3: Yellow, LED_SMD:LED_0603_1608Metric, symbol Device:LED
- added D4: Green, LED_SMD:LED_0603_1608Metric, symbol Device:LED
- added D5: Blue, LED_SMD:LED_0603_1608Metric, symbol Device:LED
- added R21, R22, R23, R24, R25: 5.1k, Resistor_SMD:R_0402_1005Metric, symbol Device:R
- JP1: renamed from JP?; footprint (none) -> Jumper:SolderJumper-2_P1.3mm_Open_Pad1.0x1.5mm
- SW1: footprint CMM2-JLC:TS-1187A-X-X-X -> ISASTM:TS-1187A-X-X-X
- gave numbers to parts that had none: 45
Connections:
- net +3V3: now also C40.1, C42.1, C44.1, C46.1, C48.1, C50.1, C52.1, C54.1, C56.1, C58.1
- net +5V: now also C41.1, C43.1, C45.1, C47.1, C49.1, C51.1, C53.1, C55.1, C57.1, C59.1
- net GND: now also C40.2, C41.2, C42.2, C43.2, C44.2, C45.2, C46.2, C47.2, C48.2, C49.2, C50.2, C51.2, C52.2, C53.2, C54.2, C55.2, C56.2, C57.2, C58.2, C59.2, R21.1, R22.1, R23.1, R24.1, R25.1
- net LV_A10: now also U1.139 (PC10)
- net LV_A11: now also U1.140 (PC11)
- net LV_A12: now also U1.141 (PC12)
- net LV_A13: now also U1.8 (PC13)
- net LV_A14: now also U1.9 (PC14)
- net LV_A15: now also U1.10 (PC15)
- net LV_A16: now also U1.7 (PI8)
- net LV_A17: now also U1.11 (PI9)
- net LV_A18: now also U1.12 (PI10)
- net LV_A19: now also U1.13 (PI11)
- net LV_A8: now also U1.117 (PC8)
- net LV_A9: now also U1.118 (PC9)
- net LV_AEN: now also U1.120 (PA9)
- net LV_ALE: now also U1.121 (PA10)
- net LV_CLK: now also U1.55 (PC5)
- net LV_DRQ1: now also U1.40 (PA0)
- net LV_DRQ2: now also U1.41 (PA1)
- net LV_DRQ3: now also U1.42 (PA2)
- net LV_IO_CH_RDY: now also U1.58 (PB2)
- net LV_IRQ2: now also U1.144 (PD2)
- net LV_IRQ3: now also U1.145 (PD3)
- net LV_IRQ4: now also U1.146 (PD4)
- net LV_IRQ5: now also U1.147 (PD5)
- net LV_IRQ6: now also U1.150 (PD6)
- net LV_IRQ7: now also U1.151 (PD7)
- net LV_ISARESET: now also U1.50 (PA4)
- net LV_TC: now also U1.54 (PC4)
- net ~IOR: now also U4.3 (A1); no longer U4.6 (A4)
- net ~IOW: now also U4.4 (A2); no longer U4.5 (A3)
- net ~LV_DACK1: now also U1.52 (PA6)
- net ~LV_DACK2: now also U1.53 (PA7)
- net ~LV_DACK3: now also U1.119 (PA8)
- net ~LV_IOR: now also U1.168 (PB9), U4.21 (B1); no longer U4.18 (B4)
- net ~LV_IOW: now also U1.167 (PB8), U4.20 (B2); no longer U4.19 (B3)
- net ~LV_IO_CH_CK: now also U1.94 (PB14)
- net ~LV_NOWS: now also U1.115 (PC6)
- net ~LV_SMEMR: now also U1.165 (PB7), U4.19 (B3); no longer U4.20 (B2)
- net ~LV_SMEMW: now also U1.164 (PB6), U4.18 (B4); no longer U4.21 (B1)
- net ~SMEMR: now also U4.5 (A3); no longer U4.4 (A2)
- net ~SMEMW: now also U4.6 (A4); no longer U4.3 (A1)
- net LED1: now reaches U1.152 (PG9)
- net LED1: now also D1.2 (A)
- net LED2: now reaches U1.153 (PG10)
- net LED2: now also D2.2 (A)
- net LED3: now reaches U1.154 (PG11)
- net LED3: now also D3.2 (A)
- net LED4: now reaches U1.155 (PG12)
- net LED4: now also D4.2 (A)
- net LED5: now reaches U1.156 (PG13)
- net LED5: now also D5.2 (A)
- new net: D1.1 (K), R21.2
- new net: D2.1 (K), R22.2
- new net: D3.1 (K), R23.2
- new net: D4.1 (K), R24.2
- new net: D5.1 (K), R25.2
Other:
- moved on the sheet: C18, C22, C29, C33, C34, J3, R26, R27, R28, R29, R30, R31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
